File: pcb_hat/lr-openauto-hat.kicad_pcb (KiCad board)
At the start: 2 copper layers, 87.4 x 56 mm, 93 parts, among them J1 Conn_01x05_Male, J10 Conn_01x05_Male, J11 Conn_01x04_Male, J2 Conn_01x04_Male, J3 Conn_01x05_Male, J4 Conn_01x02_Male, J5 Conn_01x05_Male, J6 Conn_01x02_Male, J7 Conn_01x07_Male, J8 Conn_01x02_Male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

Commit message: Transition from openauto to hudiy
Parts:
- added D13: BAT54S, Package_TO_SOT_SMD:SOT-23, F.Cu at (158.0, 90.5)
Routing:
- net /RPI_PWR_EN: track 58.9 -> 76.1 mm, vias 1 -> 2
- net +3V3: track 55.4 -> 52.7 mm
- net /ARD_OILPRESSURE: track 59.7 -> 62.1 mm
- net /ARD_IGNITION: track 62.1 -> 63.3 mm
- net GND: vias 58 -> 59
