File: pcb_hat/lr-openauto-hat.kicad_sch (KiCad schematic)
At the start: 93 parts, among them J1 Conn_01x05_Male, J10 Conn_01x05_Male, J11 Conn_01x04_Male, J2 Conn_01x04_Male, J3 Conn_01x05_Male, J4 Conn_01x02_Male, J5 Conn_01x05_Male, J6 Conn_01x02_Male, J7 Conn_01x07_Male, J8 Conn_01x02_Male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

Commit message: Transition from openauto to hudiy
Parts:
- added D13: BAT54S, Package_TO_SOT_SMD:SOT-23, symbol Diode:BAV99
Connections:
- net ARD_IGNITION: now also D13.3 (K)
- net RPI_PWR_EN: now also D13.2 (A)
- no-connect marks 5 -> 6
Other:
- note added: "Diode for keeping RPi on even when Arduino is off/reset, so it can be programmed directly from RPi without poweroff"
- moved on the sheet: C3
